File: D24V22Fx_breakout/D24V22Fx_breakout.kicad_pcb (KiCad board)
At the start: 2 copper layers, 56 x 26 mm, 20 parts, among them J1 Conn_01x03_Male, J2 Conn_01x02_Male, J3 Conn_01x03_Male, J4 Conn_01x03_Male, J5 Conn_01x03_Male, J6 Conn_01x03_Male, J7 Conn_01x02_Male, Q1 Q_NMOS_GSD, U1 Pololu_D24V22Fx

Commit message: Update for longer thing
Parts:
- removed the J5 at (159.4, 78.7)
- J3, J4: footprint Connector_PinHeader_2.54mm:PinHeader_1x03_P2.54mm_Vertical -> Connector_PinHeader_2.54mm:PinHeader_1x04_P2.54mm_Vertical
- J5: renamed from J6; footprint Connector_PinHeader_2.54mm:PinHeader_1x03_P2.54mm_Vertical -> Connector_PinHeader_2.54mm:PinHeader_1x04_P2.54mm_Horizontal
- JP1: value Default -> Jumper_3_Open
- moved J3 7.65 mm to (158.8, 76.2), turned to 0 degrees
- moved J4 5.43 mm to (161.3, 76.2), turned to 0 degrees
- moved J5 4.45 mm to (163.8, 76.2), turned to 0 degrees
- moved H2 2.00 mm to (172.0, 90.0)
- moved H3 2.00 mm to (172.0, 70.0)
- renumbered J7 to J6
Connections:
- J3 pad 2: +5V -> Earth
- J4 pad 1: Earth -> +5V
- J4 pad 3: Earth -> +5V
- J5 pad 2: +5V -> Earth
Routing:
- net +5V: track 36.1 -> 37.1 mm
- net Earth: track 80.1 -> 80.5 mm, vias 15 -> 16
Other:
- board size 56 x 26 mm -> 58 x 26 mm

Commit message: Fixing paths
Parts:
- JP1: value Jumper_3_Open -> Default
- U1: footprint matt:Pololu_D24V22Fx_THT -> pololu:Pololu_D24V22Fx_THT
Changed lines of the file:
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@@
     (add_net Earth)
+  )
+  (module pololu:Pololu_D24V22Fx_THT (layer F.Cu)
+    (at 156.6926 88.16848 90)
+    (descr "Pololu D24V22Fx series regulator footprint")
+    (fp_text reference U1 (at 8.89 -5.08 90) (layer F.SilkS)
+      (effects (font (size 1 1) (thickness 0.15)))
+    )
+    (fp_text value Pololu_D24V22Fx (at 8.89 -7.62 90) (layer F.Fab)
+      (effects (font (size 1 1) (thickness 0.15)))
+    )
+    (fp_line (start 0 0) (end 0 -17.78) (layer F.SilkS) (width 0.12))
+    (fp_line (start 0 -17.8) (end 17.8 -17.8) (layer F.SilkS) (width 0.12))
+    (fp_line (start 17.8 -17.8) (end 17.8 0) (layer F.SilkS) (width 0.12))
+    (fp_line (start 17.8 0) (end 0 0) (layer F.SilkS) (width 0.12))
+    (pad 3 thru_hole circle (at 1.27 -1.27 90) (size 1.524 1.524) (drill 1.02) (layers *.Cu *.Mask)
+      (net 5 PG))
+    (pad 2 thru_hole circle (at 3.81 -1.27 90) (size 1.524 1.524) (drill 1.02) (layers *.Cu *.Mask)
+      (net 9 EN))
+    (pad 1 thru_hole circle (at 6.35 -1.27 90) (size 1.524 1.524) (drill 1.02) (layers *.Cu *.Mask)
+      (net 4 +BATT))
+    (pad 4 thru_hole circle (at 8.89 -1.27 90) (size 1.524 1.524) (drill 1.02) (layers *.Cu *.Mask)
+      (net 6 Earth))
+    (pad 6 thru_hole circle (at 11.43 -1.27 90) (size 1.524 1.524) (drill 1.02) (layers *.Cu *.Mask)
+      (net 3 +5V))
+    (pad 5 thru_hole circle (at 1.27 -11.96 90) (size 1.524 1.524) (drill 1.02) (layers *.Cu *.Mask)
+      (net 6 Earth))
+    (pad "" np_thru_hole circle (at 15.24 -2.54 90) (size 2 2) (drill 2) (layers *.Cu *.Mask))
+    (pad "" np_thru_hole circle (at 2.3 -15.5 90) (size 2 2) (drill 2) (layers *.Cu *.Mask))
+    (model ${KIPRJMOD}/../lib/kicad-libraries/3D_models/Pololu_D24V22F12.STEP
+      (offset (xyz 8.65 9.1 2.54))
+      (scale (xyz 1 1 1))
+      (rotate (xyz -90 0 -90))
+    )
   )
   (module Connector_PinHeader_2.54mm:PinHeader_1x04_P2.54mm_Horizontal (layer F.Cu)
@@
       (effects (font (size 1 1) (thickness 0.15)))
     )
-    (fp_text value Jumper_3_Open (at 1 1.5) (layer F.SilkS)
+    (fp_text value Default (at 1 1.5) (layer F.SilkS)
       (effects (font (size 0.5 0.5) (thickness 0.1)))
     )
@@
     )
   )
-  (module matt:Pololu_D24V22Fx_THT (layer F.Cu)
-    (at 156.6926 88.16848 90)
-    (descr "Pololu D24V22Fx series regulator footprint")
-    (fp_text reference U1 (at 8.89 -5.08 90) (layer F.SilkS)
-      (effects (font (size 1 1) (thickness 0.15)))
-    )
-    (fp_text value Pololu_D24V22Fx (at 8.89 -7.62 90) (layer F.Fab)
-      (effects (font (size 1 1) (thickness 0.15)))
-    )
-    (fp_line (start 0 0) (end 0 -17.78) (layer F.SilkS) (width 0.12))
-    (fp_line (start 0 -17.8) (end 17.8 -17.8) (layer F.SilkS) (width 0.12))
-    (fp_line (start 17.8 -17.8) (end 17.8 0) (layer F.SilkS) (width 0.12))
-    (fp_line (start 17.8 0) (end 0 0) (layer F.SilkS) (width 0.12))
-    (pad 3 thru_hole circle (at 1.27 -1.27 90) (size 1.524 1.524) (drill 1.02) (layers *.Cu *.Mask)
-      (net 5 PG))
-    (pad 2 thru_hole circle (at 3.81 -1.27 90) (size 1.524 1.524) (drill 1.02) (layers *.Cu *.Mask)
-      (net 9 EN))
-    (pad 1 thru_hole circle (at 6.35 -1.27 90) (size 1.524 1.524) (drill 1.02) (layers *.Cu *.Mask)
-      (net 4 +BATT))
-    (pad 4 thru_hole circle (at 8.89 -1.27 90) (size 1.524 1.524) (drill 1.02) (layers *.Cu *.Mask)
-      (net 6 Earth))
-    (pad 6 thru_hole circle (at 11.43 -1.27 90) (size 1.524 1.524) (drill 1.02) (layers *.Cu *.Mask)
-      (net 3 +5V))
-    (pad 5 thru_hole circle (at 1.27 -11.96 90) (size 1.524 1.524) (drill 1.02) (layers *.Cu *.Mask)
-      (net 6 Earth))
-    (pad "" np_thru_hole circle (at 15.24 -2.54 90) (size 2 2) (drill 2) (layers *.Cu *.Mask))
-    (pad "" np_thru_hole circle (at 2.3 -15.5 90) (size 2 2) (drill 2) (layers *.Cu *.Mask))
-    (model C:/Users/matt/Documents/AFA/PCBs/lib/kicad/3D_models/Pololu_D24V22F12.STEP
-      (offset (xyz 8.890000000000001 8.890000000000001 2.54))
-      (scale (xyz 1 1 1))
-      (rotate (xyz -90 0 -90))
-    )
-  )
   (module Resistor_SMD:R_0805_2012Metric_Pad1.15x1.40mm_HandSolder (layer F.Cu)
     (at 143.6 90.3 180)
@@
     (pad "" thru_hole circle (at -8 -10 90) (size 1.4 1.4) (drill 1) (layers *.Cu *.Mask))
     (pad "" thru_hole circle (at 3 -10 90) (size 1.4 1.4) (drill 1) (layers *.Cu *.Mask))
-    (model C:/Users/matt/Documents/AFA/PCBs/lib/kicad/3D_models/XT30PW_male.STEP
+    (model ${KIPRJMOD}/../lib/kicad-libraries/3D_models/XT30PW_male.STEP
       (offset (xyz -2.5 4 2.5))
       (scale (xyz 1 1 1))

Commit message: Updated the silkscreen to include dimesnions
Other:
- board text added: "------> 52 mm | | (M2) | v 20 mm"
